Commit message: Fix manipulator to world is optional

File: manipulator_h_description/urdf/manipulator_h.xacro (robot description, xacro)
@@ -2,8 +2,6 @@
 <!-- Revolute-Revolute Manipulator -->
 <robot name="robotis_manipulator_h" xmlns:xacro="http://www.ros.org/wiki/xacro">
-  <!-- some parameters -->
-  <xacro:property name="pi" value="3.141592654" />
-  <!-- some parameters -->
-  <xacro:property name="pi" value="3.141592654" />
+  <!-- Configuration parameters -->
+  <xacro:arg name="fix_manipulator_h_to_world" default="true" />
   <!-- Import all Gazebo-customization elements, including Gazebo colors -->
   <xacro:include filename="$(find manipulator_h_description)/urdf/manipulator_h.gazebo" />
@@ -11,11 +9,12 @@
   <xacro:include filename="$(find manipulator_h_description)/urdf/materials.xacro" />
   <!-- Used for fixing robot to Gazebo 'link 1' -->
-  <link name="world">
-  </link>
-  <joint name="world_fixed" type="fixed">
-    <origin xyz="0 0 0" rpy="0 0 0"/>
-    <parent link="world"/>
-    <child link="link1"/>
-  </joint>
+  <xacro:if value="$(arg fix_manipulator_h_to_world)">
+    <link name="world"/>
+    <joint name="world_fixed" type="fixed">
+      <origin xyz="0 0 0" rpy="0 0 0"/>
+      <parent link="world"/>
+      <child link="link1"/>
+    </joint>
+  </xacro:if>
   <!-- link 1 -->
   <link name="link1">
